Commit message: demo test passed

File: urdf/model1-2.urdf (robot description, URDF)
Before this commit: robot model1, 6 links, 5 joints
Links:
- link base_link: geometry collision box size=0.18 0.2 0.07; visual mesh filename=file:///home/olin/Robotics/Projects/model1_workshop/src/mod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
- link bl_wheel: geometry visual mesh filename=file:///home/olin/Robotics/Projects/model1_workshop/src/mod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
- link br_wheel: geometry visual mesh filename=file:///home/olin/Robotics/Projects/model1_workshop/src/mod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
- link fl_wheel: geometry visual mesh filename=file:///home/olin/Robotics/Projects/model1_workshop/src/mod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
- link fr_wheel: geometry visual mesh filename=file:///home/olin/Robotics/Projects/model1_workshop/src/mod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
